File: besc g2.kicad_pcb (KiCad board)
At the start: 4 copper layers, 231 x 67 mm, 302 parts, among them IC1 LTC7801, J1 PHASE WIRE, J10 614105150721, J11 THROTTLE, J12 MOTOR SENSOR, J13 THROTTLE 2 (BRAKE), J14 SERIAL, J15 IGNITION, J16 CAN, J17 12V OUT, J2 PHASE WIRE, J3 PHASE WIRE, J4 BUSBAR, J5 BUSBAR, J6 IN+, J7 IN-, J8 SWD, J9 RC PWM, Q1 IRF135B203, Q10 IRF135B203, Q11 IRF135B203, Q12 IRF135B203, Q13 IRF135B203, Q14 IRF135B203, Q15 IRF135B203, Q16 IRF135B203, Q17 IRF135B203, Q18 IRF135B203, Q19 IRF135B203, Q2 IRF135B203, Q20 IRF135B203, Q21 IRF135B203, Q22 IRF135B203, Q23 IRF135B203, Q24 IRF135B203, Q25 FDMS86252L, Q26 BSC110N15NS5, Q3 IRF135B203, Q4 IRF135B203, Q5 IRF135B203, Q6 IRF135B203, Q7 IRF135B203, Q8 IRF135B203, Q9 IRF135B203, U1 UCC21520DW, U10 TJA1051T-3, U11 R-78E5.0-0.5, U12 LP5907MFX-3.3, U2 UCC21520DW, U3 UCC21520DW, U4 INA240A1D, U5 INA240A1D, U6 INA240A1D, U7 SN74LVC1G04, U8 STM32F405RGTx, U9 USBLC6-2SC6, Y1 MCSJK-7I-8.00-18-10-60-B-10

Commit message: Credits
Other:
- board text added: "Credits: github.com/vedderb github.com/galpavlin"
